Commit message: Update omni gazebo

File: omni_gazebo/urdf/omni_robot.xacro (robot description, xacro)
@@ -77,4 +77,97 @@
 		</visual>
 	</link>
+	<!-- Orbbec Astra RGBD Camera -->
+	<joint name="astra_joint" type="fixed">
+		<axis xyz="0 0 0" />
+		<origin xyz="0.15 0 0.33" rpy="0 0 0"/>
+		<parent link="base_link"/>
+		<child link="camera_link"/>
+	</joint>
+	<link name="camera_link">
+		<collision>
+			<origin xyz="0 0 0" rpy="0 0 0"/>
+			<geometry>
+				<box size="0.001 0.001 0.001"/>
+			</geometry>
+		</collision>
+		<visual>
+			<origin xyz="-0.01 0 -0.03" rpy="1.5707 0 1.5707"/>
+			<geometry>
+				<mesh filename="package://omni_gazebo/meshes/astra.dae" scale="0.001 0.001 0.001" />
+			</geometry>
+		</visual>
+		<inertial>
+			<mass value="${1e-5*scale}" />
+			<origin xyz="0 0 0" rpy="0 0 0"/>
+			<inertia ixx="0" ixy="0" ixz="0" iyy="0" iyz="0" izz="0" />
+		</inertial>
+	</link>
+	<joint name="camera_optical_joint" type="fixed">
+		<origin xyz="0 0 0" rpy="0 0 0"/>
+		<parent link="camera_link"/>
+		<child link="camera_rgb_frame"/>
+	</joint>
+	<link name="camera_rgb_frame">
+	</link>
+	<joint name="camera_depth_joint" type="fixed">
+		<origin xyz="0 0 0" rpy="-1.5707 0 -1.5707"/>
+		<parent link="camera_link"/>
+		<child link="camera_depth_frame"/>
+	</joint>
+	<link name="camera_depth_frame">
+	</link>
+	<joint name="rplidar_joint" type="fixed">
+		<axis xyz="0 1 0" />
+		<origin xyz="0.02 0 0.530" rpy="0 0 3.14"/>
+		<parent link="base_link"/>
+		<child link="laser"/>
+	</joint>
+	<!-- rplidar Laser -->
+	<link name="laser">
+		<collision>
+			<origin xyz="0 0 0" rpy="1.5707 0 4.71"/>
+			<geometry>
+				<mesh filename="package://omni_gazebo/meshes/rplidar.dae" scale="0.001 0.001 0.001" />
+			</geometry>
+		</collision>
+		<visual>
+			<origin xyz="0 0 0" rpy="1.5707 0 4.71"/>
+			<geometry>
+				<mesh filename="package://omni_gazebo/meshes/rplidar.dae" scale="0.001 0.001 0.001" />
+			</geometry>
+		</visual>
+		<inertial>
+			<mass value="${1e-5*scale}" />
+			<origin xyz="0 0 0.058" rpy="1.5707 0 4.71"/>
+			<inertia ixx="0" ixy="0" ixz="0" iyy="0" iyz="0" izz="0" />
+		</inertial>
+	</link>
+	<!-- IMU -->
+	<joint name="imu_sensor_joint" type="continuous">
+        <axis xyz="0 0 1" />
+        <origin xyz="-0.03 -0.12 0.32" rpy="0 0 0"/>
+        <parent link="base_link"/>
+        <child link="imu_link_ned"/>
+    </joint>
+    <link name="imu_link_ned">
+        <collision>
+            <origin xyz="0 0 0" rpy="0 0 0"/>
+            <geometry>
+                <box size="0.02 0.02 0.02"/>
+            </geometry>
+        </collision>
+        <visual>
+            <origin xyz="0 0 0" rpy="0 0 0"/>
+            <geometry>
+                <box size="0.02 0.02 0.02"/>
+            </geometry>
+            <material name="iRobot/Red"/>
+        </visual>
+        <inertial>
+            <mass value="${0.001*scale}" />
+            <origin xyz="0 0 0" rpy="0 0 0"/>
+            <inertia ixx="0.00000015" ixy="0" ixz="0" iyy="0.00000015" iyz="0" izz="0.00000015" />
+        </inertial>
+    </link>
 	<!-- top_wheel -->
 	<joint name="joint_top_wheel" type="fixed">

Commit message: Update omni_gazebo and create omni_control omni_fake

File: omni_gazebo/urdf/omni_robot.xacro (robot description, xacro)
@@ -144,4 +144,5 @@
 	</link>
 	<!-- IMU -->
+<!--
 	<joint name="imu_sensor_joint" type="continuous">
         <axis xyz="0 0 1" />
@@ -169,5 +170,5 @@
             <inertia ixx="0.00000015" ixy="0" ixz="0" iyy="0.00000015" iyz="0" izz="0.00000015" />
         </inertial>
-    </link>
+    </link> -->
 	<!-- top_wheel -->
 	<joint name="joint_top_wheel" type="fixed">

Commit message: Update reference and modifie omni_control

File: omni_gazebo/urdf/omni_robot.xacro (robot description, xacro)
@@ -119,5 +119,5 @@
 	<joint name="rplidar_joint" type="fixed">
 		<axis xyz="0 1 0" />
-		<origin xyz="0.02 0 0.530" rpy="0 0 3.14"/>
+		<origin xyz="0.02 0 0.530" rpy="0 0 0"/>
 		<parent link="base_link"/>
 		<child link="laser"/>
@@ -126,5 +126,5 @@
 	<link name="laser">
 		<collision>
-			<origin xyz="0 0 0" rpy="1.5707 0 4.71"/>
+			<origin xyz="0 0 0" rpy="1.5707 0 3.1412"/>
 			<geometry>
 				<mesh filename="package://omni_gazebo/meshes/rplidar.dae" scale="0.001 0.001 0.001" />
